File: Schematic/ti_based.sch (KiCad schematic (older format))
At the start: 37 parts, among them P1 HE10-10

Commit message: pcb design completed
Parts:
- removed C? (x3): CP, symbol CP
- removed D?: LED, symbol LED
- removed D?: 1N5400-E3_54, DIOAD2855W132L835D505, symbol 1N5400-E3_54
- removed IC?: ams1117-3.3v, SOT229P700X180-4N, symbol ams1117-3.3v
- removed P1: HE10-10, symbol HE10-10
- removed P?: USB_A, symbol USB_A
- removed PS?: AMS1117-5.0, SOT229P700X180-4N, symbol AMS1117-5.0
- removed R?: R, symbol R
- removed RP1: R_PACK8, symbol R_PACK8
- removed SW?: SW_PUSH, symbol SW_PUSH
- added C10, C15, C7: 0.1uF, Capacitor_SMD:C_0603_1608Metric_Pad1.05x0.95mm_HandSolder, symbol ti_based-rescue:C_Small
- added C11, C16, C27, C29, C31, C5, C9: 2.2uF, Capacitor_SMD:C_0603_1608Metric_Pad1.05x0.95mm_HandSolder, symbol Device:C
- added C12, C40, C41, C6, C8: 1uF, Capacitor_SMD:C_0603_1608Metric_Pad1.05x0.95mm_HandSolder, symbol ti_based-rescue:C_Small
- added C13, C14, C17, C18, C19, C20: 4.7nF, Capacitor_SMD:C_0603_1608Metric_Pad1.05x0.95mm_HandSolder, symbol ti_based-rescue:C_Small
- added C2, C3, C30: 10uF, Capacitor_SMD:C_0603_1608Metric_Pad1.05x0.95mm_HandSolder, symbol Device:C
- added C23: 10nF, Capacitor_SMD:C_0603_1608Metric_Pad1.05x0.95mm_HandSolder, symbol Device:C
- added C44, C45: 1uF, Capacitor_SMD:C_0603_1608Metric_Pad1.05x0.95mm_HandSolder, symbol ti_based-rescue:C
- added D1: LED, LED_SMD:LED_0603_1608Metric, symbol Device:LED
- added IC1: LM2664M6X, LM2664M6X:SOT95P280X145-6N, symbol LM2664M6X:LM2664M6X
- added IC2: TPS72325DBVT, TPS72325DBVT:SOT95P280X145-5N, symbol TPS72325DBVT:TPS72325DBVT
- added J1: Conn_01x02_Female, Connector_PinHeader_2.00mm:PinHeader_1x02_P2.00mm_Vertical, symbol Connector:Conn_01x02_Female
- added J2, J3: Conn_01x12_Female, Connector_PinHeader_2.00mm:PinHeader_1x12_P2.00mm_Vertical, symbol Connector:Conn_01x12_Female
- added R10, R11, R12, R13, R14, R3, R4, R5, R6, R7, R8, R9: 1M, Resistor_SMD:R_0603_1608Metric_Pad1.05x0.95mm_HandSolder, symbol Device:R_Small
- added R2: R, Resistor_SMD:R_0603_1608Metric_Pad1.05x0.95mm_HandSolder, symbol Device:R
- added U1: MCP1754-3302E_SOT89, MCP1754ST-3302E_MC:SON50P300X200X100-9N-D, symbol Regulator_Linear:MCP1754-3302E_SOT89
- added U2: TLV70025_SOT23-5, TLV70025DSET:SON50P150X150X80-6N, symbol Regulator_Linear:TLV70025_SOT23-5
- C1: renamed from C?; value C_Small -> 1uF; footprint (none) -> Capacitor_SMD:C_0603_1608Metric_Pad1.05x0.95mm_HandSolder; symbol C_Small -> ti_based-rescue:C_Small
- C21, C22, C24, C25, C26, C28: renamed from C?; footprint (none) -> Capacitor_SMD:C_0603_1608Metric_Pad1.05x0.95mm_HandSolder; symbol C_Small -> ti_based-rescue:C_Small
- C32, C33, C34, C35, C36, C37, C38, C39, C42, C43, C46, C47, C48, C49, C50: renamed from C?; footprint (none) -> Capacitor_SMD:C_0603_1608Metric_Pad1.05x0.95mm_HandSolder; symbol C -> ti_based-rescue:C
- C4: renamed from C?; value C_Small -> 0.1uF; footprint (none) -> Capacitor_SMD:C_0603_1608Metric_Pad1.05x0.95mm_HandSolder; symbol C_Small -> ti_based-rescue:C_Small
- IC3: renamed from IC?; footprint QFP50P1200X1200X120-64N -> ADS1299-4PAGR:QFP50P1200X1200X120-64N; symbol ADS1299-4PAGR -> ti_based-rescue:ADS1299-4PAGR
- R1: renamed from R?; footprint (none) -> Resistor_SMD:R_0603_1608Metric_Pad1.05x0.95mm_HandSolder; symbol R -> ti_based-rescue:R
Connections:
- net labels added: -RAW, AGND, AVDD, AVSS, DVDD, RAW
- net labels removed: 3.3V, 5V, CS, DRDY, Earth, GND, MISO, MOSI, PWDN, RESET, SCLK, START, VCC, VDD
- wire segments 180 -> 386
- no-connect marks 0 -> 3
Other:
- note added: "Clean +2.5V"
- note added: "Clean -2.5V"
- note removed: "AVCC/GRD"
- note removed: "AVCC\n"
- note removed: "AVDD"
- note removed: "AVDD\n"
- note removed: "AVSS"
- note removed: "AVSS\n"
- note removed: "GND"
- note removed: "Power Supply 5V/3.3V regulated\n"
- note removed: "Vcc\n"
- moved on the sheet: C1, C21, C22, C24, C25, C26, C28, C32, C4, R1
